File: hardware/rf-synthesizer.brd (EAGLE design)
At the start: 44 x 29 mm, 69 parts, among them IC1 ATMEGA168-MU, J1 U.FL, U1 ADF4351, U2 MIC5319, X1 FOX924B-10MHz, Y1 12MHz

Commit message: brd: fully routed
Parts:
- removed LED3: (no value), led:SML0805
- removed LP2: VLP-XXX-X, balto:VLP-XXX-X
- removed R5: 220, balto:0603
- added U$1: (no value), cat:CAT-L
- moved LP1 15.6 mm to (11.4, 14.5), turned to 180 degrees
- moved LED1 12.9 mm to (10.7, 14.5), turned to 270 degrees
- moved LED2 12.9 mm to (12.2, 14.5), turned to 270 degrees
- moved R13 10.4 mm to (10.1, 17.7), flipped to the top, turned to 0 degrees
- moved R15 9.75 mm to (12.8, 17.7), flipped to the top, turned to 180 degrees
- moved C1 1.86 mm to (10.4, 20.7)
- moved R22 0.91 mm to (16.9, 4.72)
- moved C10 0.76 mm to (9.60, 23.0)
- moved U2 0.76 mm to (7.62, 21.3)
- moved C25 0.76 mm to (5.64, 19.7)
- moved C5 0.55 mm to (30.6, 11.9)
- moved C4 0.55 mm to (30.6, 13.0)
- moved C6 0.48 mm to (28.0, 10.8)
- moved C7 0.48 mm to (28.0, 9.75)
- moved R21 0.46 mm to (16.9, 6.25)
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Connections:
- removed net N$16: LED3.A, R5.1
- removed net N$23: LED2.A, R15.1
- removed net RFOUT_B+: U1.14
- removed net RFOUT_B-: U1.15
- new net N$10: LED2.C, R15.2
- net GND: now also R13.1, R15.1; no longer LED1.C, LED2.C, LED3.C
- net LED_G: now also LED2.A; no longer R15.2
- net LED_R: now also LED1.A; no longer R13.2
- net MUXOUT: no longer R5.2
- net N$3: now also LED1.C, R13.2; no longer LED1.A, R13.1
Routing:
- net +3V3: track 25.0 -> 170.1 mm, vias 0 -> 14
- net RESET: track 2.24 -> 30.2 mm, vias 0 -> 3
- net SCK: track 2.31 -> 19.6 mm, vias 0 -> 1
- net CPOUT: track 4.10 -> 21.3 mm
- net CE: track 3.22 -> 18.9 mm
- net LD: track 0.86 -> 15.8 mm, vias 1 -> 2
- net MOSI: track 2.76 -> 17.5 mm, vias 0 -> 1
- net LE: track 2.99 -> 16.5 mm
- net MISO: track 0.00 -> 12.9 mm, vias 0 -> 1
- net SW: track 1.81 -> 14.7 mm
- net PDBRF: track 1.44 -> 14.3 mm, vias 1 -> 2
- net MUXOUT: track 4.06 -> 11.8 mm, vias 0 -> 2
- net LED_R: track 0.00 -> 3.12 mm
- net LED_G: track 0.00 -> 2.78 mm
- net N$3: track 0.00 -> 2.22 mm
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Other:
- board text added: "FB2015"
- board text added: "rf-synthesizer r0"

Commit message: hw: r0
Routing:
- net GND: track 23.3 -> 30.3 mm, vias 85 -> 87
- net +3V3: track 170.1 -> 170.8 mm
- net RESET: vias 3 -> 2
Other:
- board text added: "FB2016"
- board text removed: "FB2015"
Changed lines of the file:
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@@
 <board>
 <plain>
-<text x="33.6804" y="5.6388" size="1.778" layer="121">FB2015</text>
+<text x="33.6804" y="5.6388" size="1.778" layer="121">FB2016</text>
 <text x="19.05" y="27.1272" size="1.27" layer="121">rf-synthesizer r0</text>
 </plain>
@@
 <via x="11.2776" y="23.0124" extent="1-16" drill="0.3302"/>
 <via x="12.0396" y="21.1836" extent="1-16" drill="0.3302"/>
-<via x="19.9644" y="3.81" extent="1-16" drill="0.3302"/>
+<via x="20.1168" y="3.6576" extent="1-16" drill="0.3302"/>
 <via x="9.144" y="4.1148" extent="1-16" drill="0.3302"/>
 <via x="38.5572" y="17.8308" extent="1-16" drill="0.3302"/>
@@
 <via x="29.2608" y="25.146" extent="1-16" drill="0.3302"/>
 <via x="30.1752" y="24.9936" extent="1-16" drill="0.3302"/>
+<wire x1="24.0302" y1="15.8376" x2="23.0244" y2="15.8376" width="0.254" layer="1"/>
+<wire x1="23.0244" y1="15.8376" x2="22.2504" y2="16.6116" width="0.254" layer="1"/>
+<wire x1="22.2504" y1="16.6116" x2="22.2504" y2="16.764" width="0.254" layer="1"/>
+<wire x1="27.6152" y1="17.4226" x2="27.6152" y2="18.014" width="0.254" layer="1"/>
+<wire x1="27.6152" y1="18.014" x2="27.8892" y2="18.288" width="0.254" layer="1"/>
+<wire x1="27.8892" y1="18.288" x2="28.2065" y2="18.288" width="0.254" layer="1"/>
+<wire x1="28.2065" y1="18.288" x2="28.9685" y2="19.05" width="0.254" layer="1"/>
+<wire x1="14.286521875" y1="10.372875" x2="14.7828" y2="10.869153125" width="0.254" layer="1"/>
+<wire x1="14.7828" y1="10.869153125" x2="14.7828" y2="12.4968" width="0.254" layer="1"/>
+<via x="10.8204" y="21.7932" extent="1-16" drill="0.3302"/>
+<via x="17.0688" y="1.9812" extent="1-16" drill="0.3302"/>
 </signal>
 <signal name="+5V">
@@
 <wire x1="17.8308" y1="1.3716" x2="18.288" y2="1.8288" width="0.1524" layer="16"/>
 <via x="18.288" y="1.8288" extent="1-16" drill="0.3302"/>
-<wire x1="18.288" y1="1.8288" x2="20.1168" y2="1.8288" width="0.1524" layer="1"/>
-<via x="20.1168" y="1.8288" extent="1-16" drill="0.3302"/>
-<wire x1="20.1168" y1="1.8288" x2="20.8788" y2="1.0668" width="0.1524" layer="1"/>
-<wire x1="20.8788" y1="1.0668" x2="26.0604" y2="1.0668" width="0.1524" layer="1"/>
+<wire x1="18.288" y1="1.8288" x2="20.7264" y2="1.8288" width="0.1524" layer="1"/>
+<wire x1="20.7264" y1="1.8288" x2="21.4884" y2="1.0668" width="0.1524" layer="1"/>
+<wire x1="21.4884" y1="1.0668" x2="26.0604" y2="1.0668" width="0.1524" layer="1"/>
 <wire x1="26.0604" y1="1.0668" x2="27.0764" y2="2.0828" width="0.1524" layer="1"/>
 </signal>
@@
 <wire x1="18.7452" y1="0.762" x2="19.2024" y2="1.2192" width="0.6096" layer="16"/>
 <wire x1="19.2024" y1="1.2192" x2="19.6596" y2="0.762" width="0.6096" layer="16"/>
-<wire x1="19.2024" y1="11.2776" x2="19.2024" y2="9.144" width="0.6096" layer="16"/>
+<wire x1="19.2024" y1="10.8204" x2="19.2024" y2="9.144" width="0.6096" layer="16"/>
 <wire x1="19.2024" y1="9.144" x2="19.2024" y2="6.5532" width="0.6096" layer="16"/>
 <wire x1="19.2024" y1="6.5532" x2="18.8976" y2="6.2484" width="0.6096" layer="16"/>
@@
 <via x="29.1084" y="5.0292" extent="1-16" drill="0.3302"/>
 <wire x1="28.6512" y1="5.0292" x2="29.1084" y2="5.0292" width="0.6096" layer="16"/>
-<wire x1="21.9456" y1="12.8141" x2="20.7389" y2="12.8141" width="0.6096" layer="1"/>
-<wire x1="20.7389" y1="12.8141" x2="19.2024" y2="11.2776" width="0.6096" layer="1"/>
-<via x="19.2024" y="11.2776" extent="1-16" drill="0.3302"/>
+<wire x1="21.9456" y1="12.8141" x2="21.1961" y2="12.8141" width="0.6096" layer="1"/>
+<wire x1="21.1961" y1="12.8141" x2="19.2024" y2="10.8204" width="0.6096" layer="1"/>
+<via x="19.2024" y="10.8204" extent="1-16" drill="0.3302"/>
 <wire x1="16.6116" y1="10.5031" x2="17.9707" y2="9.144" width="0.6096" layer="1"/>
 <via x="19.2024" y="9.144" extent="1-16" drill="0.3302"/>
@@
 <wire x1="13.716" y1="20.2692" x2="13.716" y2="22.7076" width="0.6096" layer="16"/>
 <wire x1="13.716" y1="22.7076" x2="14.478" y2="23.4696" width="0.6096" layer="16"/>
-<wire x1="32.3088" y1="18.7452" x2="32.3088" y2="25.2984" width="0.6096" layer="16"/>
-<wire x1="32.3088" y1="25.2984" x2="29.4132" y2="28.194" width="0.6096" layer="16"/>
-<wire x1="29.4132" y1="28.194" x2="24.384" y2="28.194" width="0.6096" layer="16"/>
+<wire x1="32.3088" y1="18.7452" x2="32.3088" y2="26.9748" width="0.6096" layer="16"/>
+<wire x1="31.0896" y1="28.194" x2="24.384" y2="28.194" width="0.6096" layer="16"/>
 <wire x1="7.0229" y1="16.3068" x2="7.0104" y2="16.3193" width="0.1524" layer="1"/>
 <wire x1="7.0104" y1="16.3193" x2="7.0104" y2="17.2212" width="0.1524" layer="1"/>
@@
 <wire x1="8.6868" y1="18.4404" x2="8.0772" y2="17.8308" width="0.6096" layer="16"/>
 <wire x1="8.0772" y1="17.8308" x2="7.3152" y2="17.8308" width="0.6096" layer="16"/>
+<wire x1="31.0896" y1="28.194" x2="32.3088" y2="26.9748" width="0.6096" layer="16"/>
 </signal>
 <signal name="N$1">
@@
 <wire x1="26.3652" y1="21.4884" x2="26.0604" y2="21.1836" width="0.1524" layer="16"/>
 <wire x1="26.0604" y1="21.1836" x2="26.0604" y2="17.6784" width="0.1524" layer="16"/>
-<wire x1="26.0604" y1="17.6784" x2="24.5364" y2="16.1544" width="0.1524" layer="16"/>
-<wire x1="24.5364" y1="16.1544" x2="24.5364" y2="13.2588" width="0.1524" layer="16"/>
-<wire x1="24.5364" y1="13.2588" x2="25.908" y2="11.8872" width="0.1524" layer="16"/>
+<wire x1="26.0604" y1="17.6784" x2="24.6888" y2="16.3068" width="0.1524" layer="16"/>
+<wire x1="24.6888" y1="16.3068" x2="24.6888" y2="13.1064" width="0.1524" layer="16"/>
+<wire x1="24.6888" y1="13.1064" x2="25.908" y2="11.8872" width="0.1524" layer="16"/>
 <wire x1="25.908" y1="11.8872" x2="26.5176" y2="11.8872" width="0.1524" layer="16"/>
 </signal>
@@
 <via x="25.7556" y="25.146" extent="1-16" drill="0.3302"/>
 <wire x1="25.7556" y1="25.146" x2="25.7556" y2="17.8308" width="0.1524" layer="16"/>
-<wire x1="25.7556" y1="17.8308" x2="24.2316" y2="16.3068" width="0.1524" layer="16"/>
-<wire x1="24.2316" y1="16.3068" x2="24.2316" y2="13.1064" width="0.1524" layer="16"/>
-<wire x1="24.2316" y1="13.1064" x2="26.0604" y2="11.2776" width="0.1524" layer="16"/>
+<wire x1="25.7556" y1="17.8308" x2="24.384" y2="16.4592" width="0.1524" layer="16"/>
+<wire x1="24.384" y1="16.4592" x2="24.384" y2="12.954" width="0.1524" layer="16"/>
+<wire x1="24.384" y1="12.954" x2="26.0604" y2="11.2776" width="0.1524" layer="16"/>
 <wire x1="26.0604" y1="11.2776" x2="27.1272" y2="11.2776" width="0.1524" layer="16"/>
 <wire x1="27.1272" y1="11.2776" x2="27.7368" y2="11.8872" width="0.1524" layer="16"/>
